File: rc2014-ym2151.kicad_pcb (KiCad board)
At the start: 2 copper layers, 100 x 50 mm, 36 parts, among them CON1 SJ1-3523N, J1 Conn_01x03, P1 RC2014 BUS, U1 74HCT688, U2 YM2151, U3 YM3012, U4 NJM4556, U5 NJM4556, X1 3.579545MHz

Commit message: move version tag
Other:
- board text added: "Rev: %%version%%"
- board text removed: "Date: %%date%% Version: %%version%%"
Changed lines of the file:
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@@
   (title_block
     (title "RC2014 YM2151 sound card")
-    (date %%date%%)
+    (date "2021-11-20 12:07:43")
     (rev %%version%%)
   )
@@
     )
   )
-  (gr_text "Date: %%date%% Version: %%version%%" (at 83.4 160) (layer B.SilkS)
-    (effects (font (size 1.5 1.5) (thickness 0.3)) (justify mirror))
+  (gr_text "Rev: %%version%%" (at 160.1 160.1) (layer F.SilkS)
+    (effects (font (size 1.5 1.5) (thickness 0.3)) (justify right))
   )
   (gr_text " -OP" (at 153.9 152) (layer F.SilkS)

Commit message: Tidy schematic and readme
Parts:
- C6: value C -> 0.1uF
Changed lines of the file:
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@@
       (effects (font (size 1 1) (thickness 0.15)))
     )
-    (fp_text value C (at 1.25 2.55) (layer F.Fab)
+    (fp_text value 0.1uF (at 1.25 2.55) (layer F.Fab)
       (effects (font (size 1 1) (thickness 0.15)))
     )

Commit message: Update build script to latest released version, and PCB missed from previous commit
Parts:
- C1, C12, C2, C4: value C -> 0.1uF
- C10, C11: value C_Small -> 4.7uF
- C3: value C_Small -> 0.1uF
- C5: value CP_Small -> 4.7uF
- C7: value C_Small -> 10uF / Omit?
- C8, C9: value C_Small -> 1500pF / 3300pF
- JP2: value SolderJumper_2_Bridged -> Opamp - to GND
- JP3: value SolderJumper_2_Bridged -> Opamp + to 5V
- R1: value R -> 100 / 270
- RN1: value R_Network08 -> 10K
Changed lines of the file:
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@@
       (effects (font (size 1 1) (thickness 0.15)))
     )
-    (fp_text value C (at 1.25 2.55) (layer F.Fab)
+    (fp_text value 0.1uF (at 1.25 2.55) (layer F.Fab)
       (effects (font (size 1 1) (thickness 0.15)))
     )
@@
       (effects (font (size 1 1) (thickness 0.15)))
     )
-    (fp_text value SolderJumper_2_Bridged (at 0 1.9 90) (layer F.Fab)
+    (fp_text value "Opamp + to 5V" (at 0 1.9 90) (layer F.Fab)
       (effects (font (size 1 1) (thickness 0.15)))
     )
@@
       (effects (font (size 1 1) (thickness 0.15)))
     )
-    (fp_text value SolderJumper_2_Bridged (at 0 1.9 90) (layer F.Fab)
+    (fp_text value "Opamp - to GND" (at 0 1.9 90) (layer F.Fab)
       (effects (font (size 1 1) (thickness 0.15)))
     )
@@
       (effects (font (size 1 1) (thickness 0.15)))
     )
-    (fp_text value C_Small (at 1.25 2.55) (layer F.Fab)
+    (fp_text value 0.1uF (at 1.25 2.55) (layer F.Fab)
       (effects (font (size 1 1) (thickness 0.15)))
     )
@@
       (effects (font (size 1 1) (thickness 0.15)))
     )
-    (fp_text value CP_Small (at 1.25 5) (layer F.Fab)
+    (fp_text value 4.7uF (at 1.25 5) (layer F.Fab)
       (effects (font (size 1 1) (thickness 0.15)))
     )
@@
       (effects (font (size 1 1) (thickness 0.15)))
     )
-    (fp_text value C_Small (at 1.25 5) (layer F.Fab)
+    (fp_text value 4.7uF (at 1.25 5) (layer F.Fab)
       (effects (font (size 1 1) (thickness 0.15)))
     )
@@
       (effects (font (size 1 1) (thickness 0.15)))
     )
-    (fp_text value C_Small (at 1.25 5) (layer F.Fab)
+    (fp_text value 4.7uF (at 1.25 5) (layer F.Fab)
       (effects (font (size 1 1) (thickness 0.15)))
     )
@@
       (effects (font (size 1 1) (thickness 0.15)))
     )
-    (fp_text value R (at 3.81 1.92) (layer F.Fab)
+    (fp_text value "100 / 270" (at 3.81 1.92) (layer F.Fab)
       (effects (font (size 1 1) (thickness 0.15)))
     )
@@
       (effects (font (size 1 1) (thickness 0.15)))
     )
-    (fp_text value C_Small (at 1.25 2.55) (layer F.Fab)
+    (fp_text value "1500pF / 3300pF" (at 1.25 2.55) (layer F.Fab)
       (effects (font (size 1 1) (thickness 0.15)))
     )
@@
       (effects (font (size 1 1) (thickness 0.15)))
     )
-    (fp_text value C_Small (at 1.25 2.55) (layer F.Fab)
+    (fp_text value "1500pF / 3300pF" (at 1.25 2.55) (layer F.Fab)
       (effects (font (size 1 1) (thickness 0.15)))
     )
@@
       (effects (font (size 1 1) (thickness 0.15)))
     )
-    (fp_text value C_Small (at 1.25 2.55) (layer F.Fab)
+    (fp_text value "10uF / Omit?" (at 1.25 2.55) (layer F.Fab)
       (effects (font (size 1 1) (thickness 0.15)))
     )
@@
       (effects (font (size 1 1) (thickness 0.15)))
     )
-    (fp_text value R_Network08 (at 10.16 2.4 90) (layer F.Fab)
+    (fp_text value 10K (at 10.16 2.4 90) (layer F.Fab)
       (effects (font (size 1 1) (thickness 0.15)))
     )
@@
       (effects (font (size 1 1) (thickness 0.15)))
     )
-    (fp_text value C (at 1.25 2.5 180) (layer F.Fab)
+    (fp_text value 0.1uF (at 1.25 2.5 180) (layer F.Fab)
       (effects (font (size 1 1) (thickness 0.15)))
     )
@@
       (effects (font (size 1 1) (thickness 0.15)))
     )
-    (fp_text value C (at 1.25 2.5 180) (layer F.Fab)
+    (fp_text value 0.1uF (at 1.25 2.5 180) (layer F.Fab)
       (effects (font (size 1 1) (thickness 0.15)))
     )
@@
       (effects (font (size 1 1) (thickness 0.15)))
     )
-    (fp_text value C (at 1.25 2.5 180) (layer F.Fab)
+    (fp_text value 0.1uF (at 1.25 2.5 180) (layer F.Fab)
       (effects (font (size 1 1) (thickness 0.15)))
     )
