File: rc2014-ym2151.kicad_sch (KiCad schematic)
At the start: 27 parts, among them CON1 SJ1-3523N, J1 Debug connector, P1 RC2014 BUS, U1 74HCT688, U2 YM2151, U3 YM3012, U4 NJM4556, U5 NJM4556, X1 3.579545MHz

Commit message: kicad 9 work in progress
Parts:
- U2: footprint Package_DIP:DIP-24_W15.24mm_Socket -> Package_DIP:DIP-24_W15.24mm
- U3: footprint Package_DIP:DIP-16_W7.62mm_Socket -> Package_DIP:DIP-16_W7.62mm
- X1: footprint Package_DIP:DIP-8_W7.62mm_Socket -> Oscillator:Oscillator_DIP-8
